File: EAGLE/Zio Ultrasonic Distance Sensor.sch (EAGLE design)
At the start: 49 parts, among them J2 BM04B-SRSS-TB, J3 BM04B-SRSS-TB, Q1 847, U2 STM8L051, U3 TCT40-16T, U4 TCT40-16R

Commit message: Removes old gerbers, adds some new parts
Parts:
- added U6: LMV324, SparkFun-IC-Amplifiers:LMV324
- R1, R12, R17, R18, R19, R21, R6: value 10K ±1% -> 10k; device Discretex:R-0603 -> SparkFun-Resistors:10KOHM-0603-1/10W-1%
- R13, R16, R2: value 75K ±1% -> 75k; device Discretex:R-0603 -> SparkFun-Resistors:75KOHM-0603-1/10W-1%
- R14: value 220R ±1% -> 220; device Discretex:R-0603 -> SparkFun-Resistors:220OHM-0603-1/10W-1%
- R15: value 6.8K ±1% -> 6.8k; device Discretex:R-0603 -> SparkFun-Resistors:6.8KOHM-0603-1/10W-1%
- R22, R23: value 4.7K ±1% -> 4.7k; device Discretex:R-0603 -> SparkFun-Resistors:4.7KOHM-0603-1/10W-1%
- R5: value 3.9K ±1% -> 3.9k; device Discretex:R-0603 -> SparkFun-Resistors:3.9KOHM-0603-1/10W-1%
